File: PCB1/LNA_Filtre/V9.0/LNA_GRF2070.kicad_sch (KiCad schematic)
At the start: 15 parts, among them J1 SMA_IN, J2 SMA_OUT, J3 Conn_01x02_Pin, U1 GRF2070

Commit message: pcb2_schematic
Parts:
- removed J1: SMA_IN, Connector_Coaxial:SMA_Samtec_SMA-J-P-H-ST-EM1_EdgeMount, symbol Connector:Conn_Coaxial
- removed J2: SMA_OUT, Connector_Coaxial:SMA_Samtec_SMA-J-P-H-ST-EM1_EdgeMount, symbol Connector:Conn_Coaxial
- removed J3: Conn_01x02_Pin, Connector_PinHeader_2.54mm:PinHeader_1x02_P2.54mm_Vertical, symbol Connector:Conn_01x02_Pin
Connections:
- net sig3: now reaches C1.1
- net sig4: now reaches C6.2, L3.2

Commit message: pcb2_new
Parts:
- renumbered C1 to C44, C2 to C45, C3 to C46, C4 to C47, C5 to C48, C6 to C49, L1 to L7, L2 to L8, L3 to L9, R1 to R18, U1 to U6
Changed lines of the file:
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@@
 		(dnp no)
 		(fields_autoplaced yes)
-		(property "Reference" "L1"
+		(property "Reference" "L7"
 			(at 120.65 76.1999 0)
 			(effects
@@
 			(project "LNA_GRF2070"
 				(path "/76074578-7479-44e4-aae5-03319eb4cd87/7df40738-ad77-4c2d-874d-bfbcaef2b83e"
-					(reference "L1")
+					(reference "L7")
 					(unit 1)
 				)
@@
 		(dnp no)
 		(fields_autoplaced yes)
-		(property "Reference" "C4"
+		(property "Reference" "C47"
 			(at 144.78 76.1999 0)
 			(effects
@@
 			(project "LNA_GRF2070"
 				(path "/76074578-7479-44e4-aae5-03319eb4cd87/7df40738-ad77-4c2d-874d-bfbcaef2b83e"
-					(reference "C4")
+					(reference "C47")
 					(unit 1)
 				)
@@
 		(dnp no)
 		(fields_autoplaced yes)
-		(property "Reference" "#PWR05"
+		(property "Reference" "#PWR076"
 			(at 134.62 90.17 0)
 			(effects
@@
 			(project "LNA_GRF2070"
 				(path "/76074578-7479-44e4-aae5-03319eb4cd87/7df40738-ad77-4c2d-874d-bfbcaef2b83e"
-					(reference "#PWR05")
+					(reference "#PWR076")
 					(unit 1)
 				)
@@
 		(dnp no)
 		(fields_autoplaced yes)
-		(property "Reference" "#PWR07"
+		(property "Reference" "#PWR078"
 			(at 177.8 110.49 0)
 			(effects
@@
 			(project "LNA_GRF2070"
 				(path "/76074578-7479-44e4-aae5-03319eb4cd87/7df40738-ad77-4c2d-874d-bfbcaef2b83e"
-					(reference "#PWR07")
+					(reference "#PWR078")
 					(unit 1)
 				)
@@
 		(dnp no)
 		(fields_autoplaced yes)
-		(property "Reference" "C5"
+		(property "Reference" "C48"
 			(at 157.48 93.9799 0)
 			(effects
@@
 			(project "LNA_GRF2070"
 				(path "/76074578-7479-44e4-aae5-03319eb4cd87/7df40738-ad77-4c2d-874d-bfbcaef2b83e"
-					(reference "C5")
+					(reference "C48")
 					(unit 1)
 				)
@@
 		(on_board yes)
 		(dnp no)
-		(property "Reference" "#FLG01"
+		(property "Reference" "#FLG08"
 			(at 99.06 109.855 0)
 			(effects
@@
 			(project "LNA_GRF2070"
 				(path "/76074578-7479-44e4-aae5-03319eb4cd87/7df40738-ad77-4c2d-874d-bfbcaef2b83e"
-					(reference "#FLG01")
+					(reference "#FLG08")
 					(unit 1)
 				)
@@
 		(dnp no)
 		(fields_autoplaced yes)
-		(property "Reference" "R1"
+		(property "Reference" "R18"
 			(at 82.55 82.55 90)
 			(effects
@@
 			(project "LNA_GRF2070"
 				(path "/76074578-7479-44e4-aae5-03319eb4cd87/7df40738-ad77-4c2d-874d-bfbcaef2b83e"
-					(reference "R1")
+					(reference "R18")
 					(unit 1)
 				)
@@
 		(dnp no)
 		(fields_autoplaced yes)
-		(property "Reference" "L2"
+		(property "Reference" "L8"
 			(at 160.02 86.36 90)
 			(effects
@@
 			(project "LNA_GRF2070"
 				(path "/76074578-7479-44e4-aae5-03319eb4cd87/7df40738-ad77-4c2d-874d-bfbcaef2b83e"
-					(reference "L2")
+					(reference "L8")
 					(unit 1)
 				)
@@
 		(dnp no)
 		(fields_autoplaced yes)
-		(property "Reference" "#PWR02"
+		(property "Reference" "#PWR073"
 			(at 77.47 90.17 0)
 			(effects
@@
 			(project "LNA_GRF2070"
 				(path "/76074578-7479-44e4-aae5-03319eb4cd87/7df40738-ad77-4c2d-874d-bfbcaef2b83e"
-					(reference "#PWR02")
+					(reference "#PWR073")
 					(unit 1)
 				)
@@
 		(dnp no)
 		(fields_autoplaced yes)
-		(property "Reference" "C6"
+		(property "Reference" "C49"
 			(at 207.01 93.9799 0)
 			(effects
@@
 			(project "LNA_GRF2070"
 				(path "/76074578-7479-44e4-aae5-03319eb4cd87/7df40738-ad77-4c2d-874d-bfbcaef2b83e"
-					(reference "C6")
+					(reference "C49")
 					(unit 1)
 				)
@@
 		(dnp no)
 		(fields_autoplaced yes)
-		(property "Reference" "#PWR06"
+		(property "Reference" "#PWR077"
 			(at 153.67 109.22 0)
 			(effects
@@
 			(project "LNA_GRF2070"
 				(path "/76074578-7479-44e4-aae5-03319eb4cd87/7df40738-ad77-4c2d-874d-bfbcaef2b83e"
-					(reference "#PWR06")
+					(reference "#PWR077")
 					(unit 1)
 				)
@@
 		(dnp no)
 		(fields_autoplaced yes)
-		(property "Reference" "L3"
+		(property "Reference" "L9"
 			(at 195.58 86.36 90)
 			(effects
@@
 			(project "LNA_GRF2070"
 				(path "/76074578-7479-44e4-aae5-03319eb4cd87/7df40738-ad77-4c2d-874d-bfbcaef2b83e"
-					(reference "L3")
+					(reference "L9")
 					(unit 1)
 				)
@@
 		(dnp no)
 		(fields_autoplaced yes)
-		(property "Reference" "#PWR03"
+		(property "Reference" "#PWR074"
 			(at 101.6 114.3 0)
 			(effects
@@
 			(project "LNA_GRF2070"
 				(path "/76074578-7479-44e4-aae5-03319eb4cd87/7df40738-ad77-4c2d-874d-bfbcaef2b83e"
-					(reference "#PWR03")
+					(reference "#PWR074")
 					(unit 1)
 				)
@@
 		(dnp no)
 		(fields_autoplaced yes)
-		(property "Reference" "#PWR08"
+		(property "Reference" "#PWR079"
 			(at 203.2 107.95 0)
 			(effects
@@
 			(project "LNA_GRF2070"
 				(path "/76074578-7479-44e4-aae5-03319eb4cd87/7df40738-ad77-4c2d-874d-bfbcaef2b83e"
-					(reference "#PWR08")
+					(reference "#PWR079")
 					(unit 1)
 				)
@@
 		(dnp no)
 		(fields_autoplaced yes)
-		(property "Reference" "#PWR04"
+		(property "Reference" "#PWR075"
 			(at 119.38 73.66 0)
 			(effects
@@
 			(project "LNA_GRF2070"
 				(path "/76074578-7479-44e4-aae5-03319eb4cd87/7df40738-ad77-4c2d-874d-bfbcaef2b83e"
-					(reference "#PWR04")
+					(reference "#PWR075")
 					(unit 1)
 				)
@@
 		(on_board yes)
 		(dnp no)
-		(property "Reference" "C1"
+		(property "Reference" "C44"
 			(at 82.55 98.298 90)
 			(effects
@@
 			(project "LNA_GRF2070"
 				(path "/76074578-7479-44e4-aae5-03319eb4cd87/7df40738-ad77-4c2d-874d-bfbcaef2b83e"
-					(reference "C1")
+					(reference "C44")
 					(unit 1)
 				)
@@
 		(on_board yes)
 		(dnp no)
-		(property "Reference" "C2"
+		(property "Reference" "C45"
 			(at 126.492 93.726 90)
 			(effects
@@
 			(project "LNA_GRF2070"
 				(path "/76074578-7479-44e4-aae5-03319eb4cd87/7df40738-ad77-4c2d-874d-bfbcaef2b83e"
-					(reference "C2")
+					(reference "C45")
 					(unit 1)
 				)
@@
 		(dnp no)
 		(fields_autoplaced yes)
-		(property "Reference" "C3"
+		(property "Reference" "C46"
 			(at 132.08 76.1999 0)
 			(effects
@@
 			(project "LNA_GRF2070"
 				(path "/76074578-7479-44e4-aae5-03319eb4cd87/7df40738-ad77-4c2d-874d-bfbcaef2b83e"
-					(reference "C3")
+					(reference "C46")
 					(unit 1)
 				)
@@
 		(dnp no)
 		(fields_autoplaced yes)
-		(property "Reference" "#FLG02"
+		(property "Reference" "#FLG09"
 			(at 117.475 69.85 0)
 			(effects
@@
 			(project "LNA_GRF2070"
 				(path "/76074578-7479-44e4-aae5-03319eb4cd87/7df40738-ad77-4c2d-874d-bfbcaef2b83e"
-					(reference "#FLG02")
+					(reference "#FLG09")
 					(unit 1)
 				)
@@
 		(dnp no)
 		(fields_autoplaced yes)
-		(property "Reference" "U1"
+		(property "Reference" "U6"
 			(at 102.87 81.28 0)
 			(effects
@@
 			(project "LNA_GRF2070"
 				(path "/76074578-7479-44e4-aae5-03319eb4cd87/7df40738-ad77-4c2d-874d-bfbcaef2b83e"
-					(reference "U1")
-					(unit 1)
-				)
+					(reference "U6")
+					(unit 1)
+				)

Commit message: capa_0402
Parts:
- C44, C45, C46, C47, C48, C49: footprint Capacitor_SMD:C_0603_1608Metric -> Capacitor_SMD:C_0402_1005Metric_Pad0.74x0.62mm_HandSolder
Changed lines of the file:
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@@
 			)
 		)
-		(property "Footprint" "Capacitor_SMD:C_0603_1608Metric"
+		(property "Footprint" "Capacitor_SMD:C_0402_1005Metric_Pad0.74x0.62mm_HandSolder"
 			(at 141.9352 81.28 0)
 			(effects
@@
 			)
 		)
-		(property "Footprint" "Capacitor_SMD:C_0603_1608Metric"
+		(property "Footprint" "Capacitor_SMD:C_0402_1005Metric_Pad0.74x0.62mm_HandSolder"
 			(at 154.6352 99.06 0)
 			(effects
@@
 			)
 		)
-		(property "Footprint" "Capacitor_SMD:C_0603_1608Metric"
+		(property "Footprint" "Capacitor_SMD:C_0402_1005Metric_Pad0.74x0.62mm_HandSolder"
 			(at 202.2348 91.44 0)
 			(effects
@@
 			)
 		)
-		(property "Footprint" "Capacitor_SMD:C_0603_1608Metric"
+		(property "Footprint" "Capacitor_SMD:C_0402_1005Metric_Pad0.74x0.62mm_HandSolder"
 			(at 86.36 93.0148 0)
 			(effects
@@
 			)
 		)
-		(property "Footprint" "Capacitor_SMD:C_0603_1608Metric"
+		(property "Footprint" "Capacitor_SMD:C_0402_1005Metric_Pad0.74x0.62mm_HandSolder"
 			(at 127 90.4748 0)
 			(effects
@@
 			)
 		)
-		(property "Footprint" "Capacitor_SMD:C_0603_1608Metric"
+		(property "Footprint" "Capacitor_SMD:C_0402_1005Metric_Pad0.74x0.62mm_HandSolder"
 			(at 129.2352 81.28 0)
 			(effects
