File: PCB1/demodulateur/Démodulateur USART ASK-2026-10-17_155308/Démodulateur USART ASK.kicad_sch (KiCad schematic)
At the start: 13 parts, among them J2 Conn_Coaxial, J3 Conn_01x03_Pin, U1 AD8313xRM

Commit message: pcb2_schematic
Parts:
- removed J2: Conn_Coaxial, Connector_Coaxial:SMA_Samtec_SMA-J-P-H-ST-EM1_EdgeMount, symbol Connector:Conn_Coaxial
- removed J3: Conn_01x03_Pin, Connector_PinHeader_2.54mm:PinHeader_1x03_P2.54mm_Vertical, symbol Connector:Conn_01x03_Pin
Connections:
- net VCC_demod renamed +3.3V
- net demodIN renamed sig4
- net demodOUT renamed sig5
Other:
- note removed: "Port SMA"
- note removed: "Port d'alimentation VCC"

Commit message: pcb2_new
Parts:
- renumbered C2 to C40, C3 to C41, C1 to C42, C4 to C43, R1 to R14, R2 to R15, R4 to R16, R3 to R17, U1 to U5
Changed lines of the file:
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@@
 		(dnp no)
 		(fields_autoplaced yes)
-		(property "Reference" "#PWR07"
+		(property "Reference" "#PWR067"
 			(at 119.38 41.91 0)
 			(effects
@@
 			(project "Démodulateur USART ASK"
 				(path "/76074578-7479-44e4-aae5-03319eb4cd87/ca14d6bf-a943-4d46-b7a9-fa4078108804"
-					(reference "#PWR07")
+					(reference "#PWR067")
 					(unit 1)
 				)
@@
 		(dnp no)
 		(fields_autoplaced yes)
-		(property "Reference" "#PWR01"
+		(property "Reference" "#PWR069"
 			(at 134.62 96.52 0)
 			(effects
@@
 			(project "Démodulateur USART ASK"
 				(path "/76074578-7479-44e4-aae5-03319eb4cd87/ca14d6bf-a943-4d46-b7a9-fa4078108804"
-					(reference "#PWR01")
+					(reference "#PWR069")
 					(unit 1)
 				)
@@
 		(dnp no)
 		(fields_autoplaced yes)
-		(property "Reference" "C2"
+		(property "Reference" "C40"
 			(at 102.87 63.5 90)
 			(effects
@@
 			(project "Démodulateur USART ASK"
 				(path "/76074578-7479-44e4-aae5-03319eb4cd87/ca14d6bf-a943-4d46-b7a9-fa4078108804"
-					(reference "C2")
+					(reference "C40")
 					(unit 1)
 				)
@@
 		(dnp no)
 		(fields_autoplaced yes)
-		(property "Reference" "#PWR043"
+		(property "Reference" "#PWR072"
 			(at 167.64 58.42 0)
 			(effects
@@
 			(project "gros_pcb_commun"
 				(path "/76074578-7479-44e4-aae5-03319eb4cd87/ca14d6bf-a943-4d46-b7a9-fa4078108804"
-					(reference "#PWR043")
+					(reference "#PWR072")
 					(unit 1)
 				)
@@
 		(dnp no)
 		(fields_autoplaced yes)
-		(property "Reference" "#PWR033"
+		(property "Reference" "#PWR065"
 			(at 99.06 58.42 0)
 			(effects
@@
 			(project ""
 				(path "/76074578-7479-44e4-aae5-03319eb4cd87/ca14d6bf-a943-4d46-b7a9-fa4078108804"
-					(reference "#PWR033")
+					(reference "#PWR065")
 					(unit 1)
 				)
@@
 		(dnp no)
 		(fields_autoplaced yes)
-		(property "Reference" "R3"
+		(property "Reference" "R17"
 			(at 160.02 52.07 90)
 			(effects
@@
 			(project "Démodulateur USART ASK"
 				(path "/76074578-7479-44e4-aae5-03319eb4cd87/ca14d6bf-a943-4d46-b7a9-fa4078108804"
-					(reference "R3")
+					(reference "R17")
 					(unit 1)
 				)
@@
 		(dnp no)
 		(fields_autoplaced yes)
-		(property "Reference" "C1"
+		(property "Reference" "C42"
 			(at 123.19 50.7999 0)
 			(effects
@@
 			(project "Démodulateur USART ASK"
 				(path "/76074578-7479-44e4-aae5-03319eb4cd87/ca14d6bf-a943-4d46-b7a9-fa4078108804"
-					(reference "C1")
+					(reference "C42")
 					(unit 1)
 				)
@@
 		(dnp no)
 		(fields_autoplaced yes)
-		(property "Reference" "#FLG02"
+		(property "Reference" "#FLG07"
 			(at 139.065 62.23 0)
 			(effects
@@
 			(project "Démodulateur USART ASK"
 				(path "/76074578-7479-44e4-aae5-03319eb4cd87/ca14d6bf-a943-4d46-b7a9-fa4078108804"
-					(reference "#FLG02")
+					(reference "#FLG07")
 					(unit 1)
 				)
@@
 		(dnp no)
 		(fields_autoplaced yes)
-		(property "Reference" "#PWR04"
+		(property "Reference" "#PWR066"
 			(at 96.52 88.9 0)
 			(effects
@@
 			(project "Démodulateur USART ASK"
 				(path "/76074578-7479-44e4-aae5-03319eb4cd87/ca14d6bf-a943-4d46-b7a9-fa4078108804"
-					(reference "#PWR04")
+					(reference "#PWR066")
 					(unit 1)
 				)
@@
 		(dnp no)
 		(fields_autoplaced yes)
-		(property "Reference" "R4"
+		(property "Reference" "R16"
 			(at 156.21 77.4699 0)
 			(effects
@@
 			(project "Démodulateur USART ASK"
 				(path "/76074578-7479-44e4-aae5-03319eb4cd87/ca14d6bf-a943-4d46-b7a9-fa4078108804"
-					(reference "R4")
+					(reference "R16")
 					(unit 1)
 				)
@@
 		(dnp no)
 		(fields_autoplaced yes)
-		(property "Reference" "#PWR06"
+		(property "Reference" "#PWR071"
 			(at 167.64 91.44 0)
 			(effects
@@
 			(project "Démodulateur USART ASK"
 				(path "/76074578-7479-44e4-aae5-03319eb4cd87/ca14d6bf-a943-4d46-b7a9-fa4078108804"
-					(reference "#PWR06")
+					(reference "#PWR071")
 					(unit 1)
 				)
@@
 		(dnp no)
 		(fields_autoplaced yes)
-		(property "Reference" "C4"
+		(property "Reference" "C43"
 			(at 149.86 50.7999 0)
 			(effects
@@
 			(project "Démodulateur USART ASK"
 				(path "/76074578-7479-44e4-aae5-03319eb4cd87/ca14d6bf-a943-4d46-b7a9-fa4078108804"
-					(reference "C4")
+					(reference "C43")
 					(unit 1)
 				)
@@
 		(on_board yes)
 		(dnp no)
-		(property "Reference" "C3"
+		(property "Reference" "C41"
 			(at 102.87 87.63 90)
 			(effects
@@
 			(project "Démodulateur USART ASK"
 				(path "/76074578-7479-44e4-aae5-03319eb4cd87/ca14d6bf-a943-4d46-b7a9-fa4078108804"
-					(reference "C3")
+					(reference "C41")
 					(unit 1)
 				)
@@
 		(dnp no)
 		(fields_autoplaced yes)
-		(property "Reference" "#PWR02"
+		(property "Reference" "#PWR068"
 			(at 115.57 82.55 0)
 			(effects
@@
 			(project "Démodulateur USART ASK"
 				(path "/76074578-7479-44e4-aae5-03319eb4cd87/ca14d6bf-a943-4d46-b7a9-fa4078108804"
-					(reference "#PWR02")
+					(reference "#PWR068")
 					(unit 1)
 				)
@@
 		(on_board yes)
 		(dnp no)
-		(property "Reference" "R1"
+		(property "Reference" "R14"
 			(at 109.22 60.452 90)
 			(effects
@@
 			(project "Démodulateur USART ASK"
 				(path "/76074578-7479-44e4-aae5-03319eb4cd87/ca14d6bf-a943-4d46-b7a9-fa4078108804"
-					(reference "R1")
+					(reference "R14")
 					(unit 1)
 				)
@@
 		(dnp no)
 		(fields_autoplaced yes)
-		(property "Reference" "#PWR08"
+		(property "Reference" "#PWR070"
 			(at 146.05 41.91 0)
 			(effects
@@
 			(project "Démodulateur USART ASK"
 				(path "/76074578-7479-44e4-aae5-03319eb4cd87/ca14d6bf-a943-4d46-b7a9-fa4078108804"
-					(reference "#PWR08")
+					(reference "#PWR070")
 					(unit 1)
 				)
@@
 		(dnp no)
 		(fields_autoplaced yes)
-		(property "Reference" "#FLG01"
+		(property "Reference" "#FLG06"
 			(at 130.175 62.23 0)
 			(effects
@@
 			(project "Démodulateur USART ASK"
 				(path "/76074578-7479-44e4-aae5-03319eb4cd87/ca14d6bf-a943-4d46-b7a9-fa4078108804"
-					(reference "#FLG01")
+					(reference "#FLG06")
 					(unit 1)
 				)
@@
 		(dnp no)
 		(fields_autoplaced yes)
-		(property "Reference" "R2"
+		(property "Reference" "R15"
 			(at 115.57 74.9299 0)
 			(effects
@@
 			(project "Démodulateur USART ASK"
 				(path "/76074578-7479-44e4-aae5-03319eb4cd87/ca14d6bf-a943-4d46-b7a9-fa4078108804"
-					(reference "R2")
+					(reference "R15")
 					(unit 1)
 				)
@@
 		(dnp no)
 		(fields_autoplaced yes)
-		(property "Reference" "U1"
+		(property "Reference" "U5"
 			(at 136.7633 90.17 0)
 			(effects
@@
 			(project "Démodulateur USART ASK"
 				(path "/76074578-7479-44e4-aae5-03319eb4cd87/ca14d6bf-a943-4d46-b7a9-fa4078108804"
-					(reference "U1")
-					(unit 1)
-				)
+					(reference "U5")
+					(unit 1)
+				)

Commit message: capa_0402
Parts:
- C40, C41, C42, C43: footprint Capacitor_SMD:C_0603_1608Metric -> Capacitor_SMD:C_0402_1005Metric_Pad0.74x0.62mm_HandSolder
Changed lines of the file:
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@@
 			)
 		)
-		(property "Footprint" "Capacitor_SMD:C_0603_1608Metric"
+		(property "Footprint" "Capacitor_SMD:C_0402_1005Metric_Pad0.74x0.62mm_HandSolder"
 			(at 106.68 70.1548 0)
 			(effects
@@
 			)
 		)
-		(property "Footprint" "Capacitor_SMD:C_0603_1608Metric"
+		(property "Footprint" "Capacitor_SMD:C_0402_1005Metric_Pad0.74x0.62mm_HandSolder"
 			(at 118.4148 48.26 0)
 			(effects
@@
 			)
 		)
-		(property "Footprint" "Capacitor_SMD:C_0603_1608Metric"
+		(property "Footprint" "Capacitor_SMD:C_0402_1005Metric_Pad0.74x0.62mm_HandSolder"
 			(at 145.0848 55.88 0)
 			(effects
@@
 			)
 		)
-		(property "Footprint" "Capacitor_SMD:C_0603_1608Metric"
+		(property "Footprint" "Capacitor_SMD:C_0402_1005Metric_Pad0.74x0.62mm_HandSolder"
 			(at 106.68 80.9752 0)
 			(effects
