File: PCB1/pa_filtrage/pa_filtrage/pa_filtrage.kicad_sch (KiCad schematic)
At the start: 0 parts

Commit message: pcb_pa_filtre
Parts:
- added C1, C4, C6, C9: 0.1u, symbol Device:C_Small
- added C10, C11, C3, C8: C_Small, symbol Device:C_Small
- added C2, C5: 10u, symbol Device:C_Small
- added C7: 33p, symbol Device:C_Small
- added J1, J2, J3: Conn_Coaxial, symbol Connector:Conn_Coaxial
- added L1, L2, L3: L_Small, symbol Device:L_Small
- added R1: 5100, symbol Device:R_Small
- added U1: SKY66185-11, SKY66185-11:IC_SKY66185-11, symbol SKY66185-11:SKY66185-11
Connections:
- new net: C3.1, L1.1, U1.23 (VCC3)
- new net: C7.2, U1.4 (RFIN)
- new net: R1.2, U1.7 (~{VEN})
- new net +3.3V: C1.2, C2.2, C4.1, C5.1, C6.2, C9.1, J3.1 (In), L1.2, R1.1, U1.10 (VBIAS), U1.28 (VCC1)
- new net EXP: U1.29 (EXP), U1.29_1 (EXP), U1.29_10 (EXP), U1.29_11 (EXP), U1.29_12 (EXP), U1.29_13 (EXP), U1.29_14 (EXP), U1.29_15 (EXP), U1.29_16 (EXP), U1.29_17 (EXP), U1.29_18 (EXP), U1.29_19 (EXP), U1.29_2 (EXP), U1.29_20 (EXP), U1.29_21 (EXP), U1.29_22 (EXP), U1.29_23 (EXP), U1.29_24 (EXP), U1.29_25 (EXP), U1.29_26 (EXP), U1.29_27 (EXP), U1.29_28 (EXP), U1.29_29 (EXP), U1.29_3 (EXP), U1.29_30 (EXP), U1.29_31 (EXP), U1.29_32 (EXP), U1.29_33 (EXP), U1.29_34 (EXP), U1.29_35 (EXP), U1.29_36 (EXP), U1.29_4 (EXP), U1.29_5 (EXP), U1.29_6 (EXP), U1.29_7 (EXP), U1.29_8 (EXP), U1.29_9 (EXP)
- new net FiltreIN: C10.1, L2.1, U1.19 (RFOUT)
- new net FiltreOUT: C11.1, J2.1 (In), L3.2
- new net GND: C1.1, C10.2, C11.2, C2.1, C3.2, C4.2, C5.2, C6.1, C8.1, C9.2, J1.2 (Ext), J2.2 (Ext), J3.2 (Ext), U1.1 (GND), U1.11 (GND), U1.13 (GND), U1.15 (GND), U1.16 (GND), U1.2 (GND), U1.20 (GND), U1.21 (GND), U1.25 (GND), U1.27 (GND), U1.6 (GND)
- new net RFIN: C7.1, C8.2, J1.1 (In)
- no-connect marks 0 -> 2

Commit message: schematic_pa_filtrage
Parts:
- removed C3, C8: C_Small, symbol Device:C_Small
- removed J3: Conn_Coaxial, symbol Connector:Conn_Coaxial
- removed L1: L_Small, symbol Device:L_Small
- added J4: Conn_01x02_Pin, Connector_PinHeader_2.54mm:PinHeader_1x02_P2.54mm_Vertical, symbol Connector:Conn_01x02_Pin
- added SF1: ~, SF2425E:SF2425E, symbol import_compo:SF2425E
- C1, C2, C4, C5, C6, C7, C9: footprint (none) -> Capacitor_SMD:C_0603_1608Metric
- C10: value C_Small -> 2.7p; footprint (none) -> Capacitor_SMD:C_0603_1608Metric
- C11: value C_Small -> 3.5p; footprint (none) -> Capacitor_SMD:C_0603_1608Metric
- J1, J2: footprint (none) -> Connector_Coaxial:SMA_Samtec_SMA-J-P-H-ST-EM1_EdgeMount
- L2, L3: value L_Small -> 24n; footprint (none) -> Inductor_SMD:L_0603_1608Metric
- R1: value 5100 -> 5k1; footprint (none) -> Resistor_SMD:R_0603_1608Metric
Connections:
- net +3.3V: now also U1.23 (VCC3), J4.2 (Pin_2)
- net GND: now also J4.1 (Pin_1), SF1.1 (IN_GND), SF1.3 (GND), SF1.4 (GND), SF1.5 (OUT_GND), SF1.7 (GND), SF1.8 (GND)
- net at L3.1: now also SF1.6 (OUT)
- net at L2.2: now also SF1.2 (IN)
Other:
- moved on the sheet: C10, C11, J1, J2, L2, L3

Commit message: pa_filtre_routage
Connections:
- net +3.3V renamed 3.3V

Commit message: PCB1 fini à valider
Parts:
- removed SF1: ~, SF2425E:SF2425E, symbol import_compo:SF2425E
- added SF1: ~, SF2425E:SF2425E, symbol projet-sys-uart:SF2425E
- renumbered J4 to J3
Connections:
- net GND: now also SF1.1 (IN_GND), SF1.3 (GND), SF1.4 (GND), SF1.5 (OUT_GND), SF1.7 (GND), SF1.8 (GND)
- net at L3.1: now also SF1.6 (OUT)
- net at L2.2: now also SF1.2 (IN)
- net 3.3V renamed +3.3V
Other:
- moved on the sheet: C1, C2, C4, C5, C6, C7, C9, J3, R1

Commit message: pcb2_schematic
Parts:
- removed J1, J2: Conn_Coaxial, Connector_Coaxial:SMA_Samtec_SMA-J-P-H-ST-EM1_EdgeMount, symbol Connector:Conn_Coaxial
- removed J3: Conn_01x02_Pin, Connector_PinHeader_2.54mm:PinHeader_1x02_P2.54mm_Vertical, symbol Connector:Conn_01x02_Pin
Connections:
- net FiltreOUT renamed sig2
- net RFIN renamed sig1
Other:
- moved on the sheet: C10, C11, L2, L3, SF1

Commit message: pcb2_new
Parts:
- renumbered C6 to C29, C10 to C30, C7 to C31, C1 to C32, C2 to C33, C11 to C34, C9 to C35, C4 to C36, C5 to C37, L2 to L4, L3 to L5, R1 to R10, U1 to U3
Changed lines of the file:
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@@
 		(dnp no)
 		(fields_autoplaced yes)
-		(property "Reference" "#PWR021"
+		(property "Reference" "#PWR047"
 			(at 96.52 68.58 0)
 			(effects
@@
 			(project "pa_filtrage"
 				(path "/76074578-7479-44e4-aae5-03319eb4cd87/77eba17e-8242-4bd9-8345-27323023ef6f"
-					(reference "#PWR021")
+					(reference "#PWR047")
 					(unit 1)
 				)
@@
 		(on_board yes)
 		(dnp no)
-		(property "Reference" "#PWR08"
+		(property "Reference" "#PWR045"
 			(at 78.74 120.65 0)
 			(effects
@@
 			(project ""
 				(path "/76074578-7479-44e4-aae5-03319eb4cd87/77eba17e-8242-4bd9-8345-27323023ef6f"
-					(reference "#PWR08")
+					(reference "#PWR045")
 					(unit 1)
 				)
@@
 		(dnp no)
 		(fields_autoplaced yes)
-		(property "Reference" "C5"
+		(property "Reference" "C37"
 			(at 167.64 105.4162 0)
 			(effects
@@
 			(project "pa_filtrage"
 				(path "/76074578-7479-44e4-aae5-03319eb4cd87/77eba17e-8242-4bd9-8345-27323023ef6f"
-					(reference "C5")
+					(reference "C37")
 					(unit 1)
 				)
@@
 		(dnp no)
 		(fields_autoplaced yes)
-		(property "Reference" "C9"
+		(property "Reference" "C35"
 			(at 143.51 109.2262 0)
 			(effects
@@
 			(project ""
 				(path "/76074578-7479-44e4-aae5-03319eb4cd87/77eba17e-8242-4bd9-8345-27323023ef6f"
-					(reference "C9")
+					(reference "C35")
 					(unit 1)
 				)
@@
 		(dnp no)
 		(fields_autoplaced yes)
-		(property "Reference" "C7"
+		(property "Reference" "C31"
 			(at 80.0163 105.41 90)
 			(effects
@@
 			(project ""
 				(path "/76074578-7479-44e4-aae5-03319eb4cd87/77eba17e-8242-4bd9-8345-27323023ef6f"
-					(reference "C7")
+					(reference "C31")
 					(unit 1)
 				)
@@
 		(dnp no)
 		(fields_autoplaced yes)
-		(property "Reference" "L3"
+		(property "Reference" "L5"
 			(at 132.08 52.07 90)
 			(effects
@@
 			(project "pa_filtrage"
 				(path "/76074578-7479-44e4-aae5-03319eb4cd87/77eba17e-8242-4bd9-8345-27323023ef6f"
-					(reference "L3")
+					(reference "L5")
 					(unit 1)
 				)
@@
 		(dnp no)
 		(fields_autoplaced yes)
-		(property "Reference" "#PWR07"
+		(property "Reference" "#PWR043"
 			(at 62.23 116.84 0)
 			(effects
@@
 			(project ""
 				(path "/76074578-7479-44e4-aae5-03319eb4cd87/77eba17e-8242-4bd9-8345-27323023ef6f"
-					(reference "#PWR07")
+					(reference "#PWR043")
 					(unit 1)
 				)
@@
 		(dnp no)
 		(fields_autoplaced yes)
-		(property "Reference" "#PWR012"
+		(property "Reference" "#PWR044"
 			(at 77.47 71.12 0)
 			(effects
@@
 			(project ""
 				(path "/76074578-7479-44e4-aae5-03319eb4cd87/77eba17e-8242-4bd9-8345-27323023ef6f"
-					(reference "#PWR012")
+					(reference "#PWR044")
 					(unit 1)
 				)
@@
 		(dnp no)
 		(fields_autoplaced yes)
-		(property "Reference" "#PWR09"
+		(property "Reference" "#PWR056"
 			(at 140.97 119.38 0)
 			(effects
@@
 			(project ""
 				(path "/76074578-7479-44e4-aae5-03319eb4cd87/77eba17e-8242-4bd9-8345-27323023ef6f"
-					(reference "#PWR09")
+					(reference "#PWR056")
 					(unit 1)
 				)
@@
 		(on_board yes)
 		(dnp no)
-		(property "Reference" "#PWR019"
+		(property "Reference" "#PWR055"
 			(at 137.16 106.68 0)
 			(effects
@@
 			(project "pa_filtrage"
 				(path "/76074578-7479-44e4-aae5-03319eb4cd87/77eba17e-8242-4bd9-8345-27323023ef6f"
-					(reference "#PWR019")
+					(reference "#PWR055")
 					(unit 1)
 				)
@@
 		(dnp no)
 		(fields_autoplaced yes)
-		(property "Reference" "U1"
+		(property "Reference" "U3"
 			(at 106.68 93.98 0)
 			(effects
@@
 			(project ""
 				(path "/76074578-7479-44e4-aae5-03319eb4cd87/77eba17e-8242-4bd9-8345-27323023ef6f"
-					(reference "U1")
+					(reference "U3")
 					(unit 1)
 				)
@@
 		(dnp no)
 		(fields_autoplaced yes)
-		(property "Reference" "#PWR05"
+		(property "Reference" "#PWR058"
 			(at 165.1 115.57 0)
 			(effects
@@
 			(project ""
 				(path "/76074578-7479-44e4-aae5-03319eb4cd87/77eba17e-8242-4bd9-8345-27323023ef6f"
-					(reference "#PWR05")
+					(reference "#PWR058")
 					(unit 1)
 				)
@@
 		(dnp no)
 		(fields_autoplaced yes)
-		(property "Reference" "L2"
+		(property "Reference" "L4"
 			(at 86.36 49.53 90)
 			(effects
@@
 			(project ""
 				(path "/76074578-7479-44e4-aae5-03319eb4cd87/77eba17e-8242-4bd9-8345-27323023ef6f"
-					(reference "L2")
+					(reference "L4")
 					(unit 1)
 				)
@@
 		(dnp no)
 		(fields_autoplaced yes)
-		(property "Reference" "#PWR02"
+		(property "Reference" "#PWR052"
 			(at 137.16 87.63 0)
 			(effects
@@
 			(project ""
 				(path "/76074578-7479-44e4-aae5-03319eb4cd87/77eba17e-8242-4bd9-8345-27323023ef6f"
-					(reference "#PWR02")
+					(reference "#PWR052")
 					(unit 1)
 				)
@@
 		(dnp no)
 		(fields_autoplaced yes)
-		(property "Reference" "#PWR01"
+		(property "Reference" "#PWR050"
 			(at 127 87.63 0)
 			(effects
@@
 			(project ""
 				(path "/76074578-7479-44e4-aae5-03319eb4cd87/77eba17e-8242-4bd9-8345-27323023ef6f"
-					(reference "#PWR01")
+					(reference "#PWR050")
 					(unit 1)
 				)
@@
 		(dnp no)
 		(fields_autoplaced yes)
-		(property "Reference" "C1"
+		(property "Reference" "C32"
 			(at 129.54 95.2562 0)
 			(effects
@@
 			(project ""
 				(path "/76074578-7479-44e4-aae5-03319eb4cd87/77eba17e-8242-4bd9-8345-27323023ef6f"
-					(reference "C1")
+					(reference "C32")
 					(unit 1)
 				)
@@
 		(dnp no)
 		(fields_autoplaced yes)
-		(property "Reference" "#PWR014"
+		(property "Reference" "#PWR048"
 			(at 119.38 41.91 0)
 			(effects
@@
 			(project "pa_filtrage"
 				(path "/76074578-7479-44e4-aae5-03319eb4cd87/77eba17e-8242-4bd9-8345-27323023ef6f"
-					(reference "#PWR014")
+					(reference "#PWR048")
 					(unit 1)
 				)
@@
 		(dnp no)
 		(fields_autoplaced yes)
-		(property "Reference" "#PWR04"
+		(property "Reference" "#PWR057"
 			(at 154.94 115.57 0)
 			(effects
@@
 			(project ""
 				(path "/76074578-7479-44e4-aae5-03319eb4cd87/77eba17e-8242-4bd9-8345-27323023ef6f"
-					(reference "#PWR04")
+					(reference "#PWR057")
 					(unit 1)
 				)
@@
 		(dnp no)
 		(fields_autoplaced yes)
-		(property "Reference" "C2"
+		(property "Reference" "C33"
 			(at 139.7 95.2562 0)
 			(effects
@@
 			(project ""
 				(path "/76074578-7479-44e4-aae5-03319eb4cd87/77eba17e-8242-4bd9-8345-27323023ef6f"
-					(reference "C2")
+					(reference "C33")
 					(unit 1)
 				)
@@
 		(dnp no)
 		(fields_autoplaced yes)
-		(property "Reference" "#PWR015"
+		(property "Reference" "#PWR046"
 			(at 96.52 41.91 0)
 			(effects
@@
 			(project "pa_filtrage"
 				(path "/76074578-7479-44e4-aae5-03319eb4cd87/77eba17e-8242-4bd9-8345-27323023ef6f"
-					(reference "#PWR015")
+					(reference "#PWR046")
 					(unit 1)
 				)
@@
 		(dnp no)
 		(fields_autoplaced yes)
-		(property "Reference" "C4"
+		(property "Reference" "C36"
 			(at 157.48 105.4162 0)
 			(effects
@@
 			(project "pa_filtrage"
 				(path "/76074578-7479-44e4-aae5-03319eb4cd87/77eba17e-8242-4bd9-8345-27323023ef6f"
-					(reference "C4")
+					(reference "C36")
 					(unit 1)
 				)
@@
 		(dnp no)
 		(fields_autoplaced yes)
-		(property "Reference" "#PWR016"
+		(property "Reference" "#PWR049"
 			(at 119.38 68.58 0)
 			(effects
@@
 			(project "pa_filtrage"
 				(path "/76074578-7479-44e4-aae5-03319eb4cd87/77eba17e-8242-4bd9-8345-27323023ef6f"
-					(reference "#PWR016")
+					(reference "#PWR049")
 					(unit 1)
 				)
@@
 		(on_board yes)
 		(dnp no)
-		(property "Reference" "#PWR017"
+		(property "Reference" "#PWR053"
 			(at 133.35 101.6 0)
 			(effects
@@
 			(project "pa_filtrage"
 				(path "/76074578-7479-44e4-aae5-03319eb4cd87/77eba17e-8242-4bd9-8345-27323023ef6f"
-					(reference "#PWR017")
+					(reference "#PWR053")
 					(unit 1)
 				)
@@
 		(dnp no)
 		(fields_autoplaced yes)
-		(property "Reference" "#PWR06"
+		(property "Reference" "#PWR051"
 			(at 133.35 121.92 0)
 			(effects
@@
 			(project ""
 				(path "/76074578-7479-44e4-aae5-03319eb4cd87/77eba17e-8242-4bd9-8345-27323023ef6f"
-					(reference "#PWR06")
+					(reference "#PWR051")
 					(unit 1)
 				)
@@
 		(on_board yes)
 		(dnp no)
-		(property "Reference" "#PWR018"
+		(property "Reference" "#PWR059"
 			(at 166.37 104.14 0)
 			(effects
@@
 			(project "pa_filtrage"
 				(path "/76074578-7479-44e4-aae5-03319eb4cd87/77eba17e-8242-4bd9-8345-27323023ef6f"
-					(reference "#PWR018")
+					(reference "#PWR059")
 					(unit 1)
 				)
@@
 		(dnp no)
 		(fields_autoplaced yes)
-		(property "Reference" "C10"
+		(property "Reference" "C30"
 			(at 80.01 58.4262 0)
 			(effects
@@
 			(project ""
 				(path "/76074578-7479-44e4-aae5-03319eb4cd87/77eba17e-8242-4bd9-8345-27323023ef6f"
-					(reference "C10")
+					(reference "C30")
 					(unit 1)
 				)
@@
 		(dnp no)
 		(fields_autoplaced yes)
-		(property "Reference" "#PWR013"
+		(property "Reference" "#PWR054"
 			(at 139.7 71.12 0)
 			(effects
@@
 			(project "pa_filtrage"
 				(path "/76074578-7479-44e4-aae5-03319eb4cd87/77eba17e-8242-4bd9-8345-27323023ef6f"
-					(reference "#PWR013")
+					(reference "#PWR054")
 					(unit 1)
 				)
@@
 		(on_board yes)
 		(dnp no)
-		(property "Reference" "R1"
+		(property "Reference" "R10"
 			(at 84.074 121.158 90)
 			(effects
@@
 			(project ""
 				(path "/76074578-7479-44e4-aae5-03319eb4cd87/77eba17e-8242-4bd9-8345-27323023ef6f"
-					(reference "R1")
+					(reference "R10")
 					(unit 1)
 				)
@@
 		(on_board yes)
 		(dnp no)
-		(property "Reference" "C6"
+		(property "Reference" "C29"
 			(at 74.93 122.428 90)
 			(effects
@@
 			(project ""
 				(path "/76074578-7479-44e4-aae5-03319eb4cd87/77eba17e-8242-4bd9-8345-27323023ef6f"
-					(reference "C6")
+					(reference "C29")
 					(unit 1)
 				)
@@
 		(dnp no)
 		(fields_autoplaced yes)
-		(property "Reference" "C11"
+		(property "Reference" "C34"
 			(at 142.24 60.9662 0)
 			(effects
@@
 			(project "pa_filtrage"
 				(path "/76074578-7479-44e4-aae5-03319eb4cd87/77eba17e-8242-4bd9-8345-27323023ef6f"
-					(reference "C11")
-					(unit 1)
-				)
+					(reference "C34")
+					(unit 1)
+				)

Commit message: capa_0402
Parts:
- C29, C30, C31, C32, C34, C35, C36: footprint Capacitor_SMD:C_0603_1608Metric -> Capacitor_SMD:C_0402_1005Metric_Pad0.74x0.62mm_HandSolder
- C33, C37: footprint Capacitor_SMD:C_0603_1608Metric -> Capacitor_SMD:C_0603_1608Metric_Pad1.08x0.95mm_HandSolder
Changed lines of the file:
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@@
 			)
 		)
-		(property "Footprint" "Capacitor_SMD:C_0603_1608Metric"
+		(property "Footprint" "Capacitor_SMD:C_0603_1608Metric_Pad1.08x0.95mm_HandSolder"
 			(at 165.1 106.68 0)
 			(effects
@@
 			)
 		)
-		(property "Footprint" "Capacitor_SMD:C_0603_1608Metric"
+		(property "Footprint" "Capacitor_SMD:C_0402_1005Metric_Pad0.74x0.62mm_HandSolder"
 			(at 140.97 110.49 0)
 			(effects
@@
 			)
 		)
-		(property "Footprint" "Capacitor_SMD:C_0603_1608Metric"
+		(property "Footprint" "Capacitor_SMD:C_0402_1005Metric_Pad0.74x0.62mm_HandSolder"
 			(at 80.01 111.76 0)
 			(effects
@@
 			)
 		)
-		(property "Footprint" "Capacitor_SMD:C_0603_1608Metric"
+		(property "Footprint" "Capacitor_SMD:C_0402_1005Metric_Pad0.74x0.62mm_HandSolder"
 			(at 127 96.52 0)
 			(effects
@@
 			)
 		)
-		(property "Footprint" "Capacitor_SMD:C_0603_1608Metric"
+		(property "Footprint" "Capacitor_SMD:C_0603_1608Metric_Pad1.08x0.95mm_HandSolder"
 			(at 137.16 96.52 0)
 			(effects
@@
 			)
 		)
-		(property "Footprint" "Capacitor_SMD:C_0603_1608Metric"
+		(property "Footprint" "Capacitor_SMD:C_0402_1005Metric_Pad0.74x0.62mm_HandSolder"
 			(at 154.94 106.68 0)
 			(effects
@@
 			)
 		)
-		(property "Footprint" "Capacitor_SMD:C_0603_1608Metric"
+		(property "Footprint" "Capacitor_SMD:C_0402_1005Metric_Pad0.74x0.62mm_HandSolder"
 			(at 77.47 59.69 0)
 			(effects
@@
 			)
 		)
-		(property "Footprint" "Capacitor_SMD:C_0603_1608Metric"
+		(property "Footprint" "Capacitor_SMD:C_0402_1005Metric_Pad0.74x0.62mm_HandSolder"
 			(at 74.93 116.84 0)
 			(effects
@@
 			)
 		)
-		(property "Footprint" "Capacitor_SMD:C_0603_1608Metric"
+		(property "Footprint" "Capacitor_SMD:C_0402_1005Metric_Pad0.74x0.62mm_HandSolder"
 			(at 139.7 62.23 0)
 			(effects
