File: PCB1/pa_filtrage/pa_filtrage/pa_filtrage.kicad_sch (KiCad schematic)
At the start: 14 parts, among them U3 SKY66185-11

Commit message: pcb2
Parts:
- C31: footprint Capacitor_SMD:C_0402_1005Metric_Pad0.74x0.62mm_HandSolder -> Capacitor_SMD:C_0603_1608Metric_Pad1.08x0.95mm_HandSolder
Changed lines of the file:
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@@
 			)
 		)
-		(property "Footprint" "Capacitor_SMD:C_0402_1005Metric_Pad0.74x0.62mm_HandSolder"
+		(property "Footprint" "Capacitor_SMD:C_0603_1608Metric_Pad1.08x0.95mm_HandSolder"
 			(at 80.01 111.76 0)
 			(effects
