File: PCB2/gros_pcb_commun/gros_pcb_commun.kicad_sch (KiCad schematic)
At the start: 0 parts

Commit message: pcb2
Other:
- added sheet Amplificateur de puissance Filtrage (../../PCB1/pa_filtrage/pa_filtrage/pa_filtrage.kicad_sch)
- added sheet Antenne Switch (../../PCB1/antenne_switch/switch_antenne_pcb_projet.kicad_sch)
- added sheet Démodulateur (../../PCB1/demodulateur/Démodulateur USART ASK-2026-10-17_155308/Démodulateur USART ASK.kicad_sch)
- added sheet Modulateur (../../PCB1/ASK_Mod+PLL_Oscill/ASK_Mod+PLL_Oscill.kicad_sch)
Changed lines of the file:
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@@
 	(generator_version "9.0")
 	(paper "A4")
+	(sheet
+		(at 189.23 22.86)
+		(size 52.07 40.64)
+		(exclude_from_sim no)
+		(in_bom yes)
+		(on_board yes)
+		(dnp no)
+		(fields_autoplaced yes)
+		(stroke
+			(width 0.1524)
+			(type solid)
+		)
+		(fill
+			(color 0 0 0 0.0000)
+		)
+		(property "Sheetname" "Antenne Switch"
+			(at 189.23 22.1484 0)
+			(effects
+				(font
+					(size 1.27 1.27)
+				)
+				(justify left bottom)
+			)
+		)
+		(property "Sheetfile" "../../PCB1/antenne_switch/switch_antenne_pcb_projet.kicad_sch"
+			(at 189.23 64.0846 0)
+			(effects
+				(font
+					(size 1.27 1.27)
+				)
+				(justify left top)
+			)
+		)
+		(instances
+			(project "gros_pcb_commun"
+				(path "/76074578-7479-44e4-aae5-03319eb4cd87"
+					(page "4")
+				)
+			)
+		)
+	)
+	(sheet
+		(at 105.41 22.86)
+		(size 48.26 39.37)
+		(exclude_from_sim no)
+		(in_bom yes)
+		(on_board yes)
+		(dnp no)
+		(fields_autoplaced yes)
+		(stroke
+			(width 0.1524)
+			(type solid)
+		)
+		(fill
+			(color 0 0 0 0.0000)
+		)
+		(property "Sheetname" "Amplificateur de puissance Filtrage"
+			(at 105.41 22.1484 0)
+			(effects
+				(font
+					(size 1.27 1.27)
+				)
+				(justify left bottom)
+			)
+		)
+		(property "Sheetfile" "../../PCB1/pa_filtrage/pa_filtrage/pa_filtrage.kicad_sch"
+			(at 105.41 62.8146 0)
+			(effects
+				(font
+					(size 1.27 1.27)
+				)
+				(justify left top)
+			)
+		)
+		(instances
+			(project "gros_pcb_commun"
+				(path "/76074578-7479-44e4-aae5-03319eb4cd87"
+					(page "3")
+				)
+			)
+		)
+	)
+	(sheet
+		(at 26.67 100.33)
+		(size 67.31 39.37)
+		(exclude_from_sim no)
+		(in_bom yes)
+		(on_board yes)
+		(dnp no)
+		(fields_autoplaced yes)
+		(stroke
+			(width 0.1524)
+			(type solid)
+		)
+		(fill
+			(color 0 0 0 0.0000)
+		)
+		(property "Sheetname" "Démodulateur"
+			(at 26.67 99.6184 0)
+			(effects
+				(font
+					(size 1.27 1.27)
+				)
+				(justify left bottom)
+			)
+		)
+		(property "Sheetfile" "../../PCB1/demodulateur/Démodulateur USART ASK-2026-10-17_155308/Démodulateur USART ASK.kicad_sch"
+			(at 26.67 140.2846 0)
+			(effects
+				(font
+					(size 1.27 1.27)
+				)
+				(justify left top)
+			)
+		)
+		(instances
+			(project "gros_pcb_commun"
+				(path "/76074578-7479-44e4-aae5-03319eb4cd87"
+					(page "5")
+				)
+			)
+		)
+	)
+	(sheet
+		(at 26.67 22.86)
+		(size 46.99 39.37)
+		(exclude_from_sim no)
+		(in_bom yes)
+		(on_board yes)
+		(dnp no)
+		(fields_autoplaced yes)
+		(stroke
+			(width 0.1524)
+			(type solid)
+		)
+		(fill
+			(color 0 0 0 0.0000)
+		)
+		(property "Sheetname" "Modulateur"
+			(at 26.67 22.1484 0)
+			(effects
+				(font
+					(size 1.27 1.27)
+				)
+				(justify left bottom)
+			)
+		)
+		(property "Sheetfile" "../../PCB1/ASK_Mod+PLL_Oscill/ASK_Mod+PLL_Oscill.kicad_sch"
+			(at 26.67 62.8146 0)
+			(effects
+				(font
+					(size 1.27 1.27)
+				)
+				(justify left top)
+			)
+		)
+		(instances
+			(project "gros_pcb_commun"
+				(path "/76074578-7479-44e4-aae5-03319eb4cd87"
+					(page "3")
+				)
+			)
+		)
+	)
 	(sheet_instances
 		(path "/"

Commit message: pcb2
Other:
- added sheet Amplificateur faible bruit Filtrage (untitled.kicad_sch)
Changed lines of the file:
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@@
+	)
+	(sheet
+		(at 175.26 99.06)
+		(size 72.39 44.45)
+		(exclude_from_sim no)
+		(in_bom yes)
+		(on_board yes)
+		(dnp no)
+		(fields_autoplaced yes)
+		(stroke
+			(width 0.1524)
+			(type solid)
+		)
+		(fill
+			(color 0 0 0 0.0000)
+		)
+		(property "Sheetname" "Amplificateur faible bruit Filtrage"
+			(at 175.26 98.3484 0)
+			(effects
+				(font
+					(size 1.27 1.27)
+				)
+				(justify left bottom)
+			)
+		)
+		(property "Sheetfile" "untitled.kicad_sch"
+			(at 175.26 144.0946 0)
+			(effects
+				(font
+					(size 1.27 1.27)
+				)
+				(justify left top)
+			)
+		)
+		(instances
+			(project "gros_pcb_commun"
+				(path "/76074578-7479-44e4-aae5-03319eb4cd87"
+					(page "6")
+				)
+			)
+		)
 	)
 	(sheet

Commit message: pcb2_schematic
Parts:
- added H1, H2, H3, H4: MountingHole_Pad, MountingHole:MountingHole_3.2mm_M3_Pad, symbol Mechanical:MountingHole_Pad
- added J4: Conn_01x03_Pin, symbol Connector:Conn_01x03_Pin
- added J5: Conn_01x04_Pin, symbol Connector:Conn_01x04_Pin
Connections:
- new net +2V5: J5.3 (Pin_3)
- new net +3.3V: J5.2 (Pin_2)
- new net +5V: J5.1 (Pin_1)
- new net GND: H1.1, H2.1, H3.1, H4.1, J4.3 (Pin_3), J5.4 (Pin_4)
- new net sig0: J4.1 (Pin_1)
- new net sig5: J4.2 (Pin_2)
Other:
- sheet Amplificateur de puissance Filtrage ports: added sig1, sig2; removed none
- sheet Amplificateur faible bruit Filtrage: file untitled.kicad_sch -> ../../PCB1/LNA_Filtre/V9.0/LNA_GRF2070.kicad_sch
- sheet Amplificateur faible bruit Filtrage ports: added sig3, sig4; removed none
- sheet Antenne Switch ports: added sig2, sig3; removed none
- sheet Démodulateur ports: added sig4, sig5; removed none
- sheet Modulateur ports: added sig0, sig1; removed none

Commit message: pcb2_new
Parts:
- renumbered H4 to H1, H3 to H2, H2 to H3, H1 to H4, J4 to J1, J5 to J2
Other:
- moved on the sheet: H1, H2, H3, H4, J1, J2

Commit message: capa_0402
Parts:
- J1: footprint (none) -> Connector_PinHeader_2.54mm:PinHeader_1x03_P2.54mm_Vertical
- J2: footprint (none) -> Connector_PinHeader_2.54mm:PinHeader_1x04_P2.54mm_Vertical
Changed lines of the file:
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@@
 			)
 		)
-		(property "Footprint" ""
+		(property "Footprint" "Connector_PinHeader_2.54mm:PinHeader_1x04_P2.54mm_Vertical"
 			(at 39.37 35.56 0)
 			(effects
@@
 			)
 		)
-		(property "Footprint" ""
+		(property "Footprint" "Connector_PinHeader_2.54mm:PinHeader_1x03_P2.54mm_Vertical"
 			(at 38.1 72.39 0)
 			(effects
