File: PCB2/gros_pcb_commun/gros_pcb_commun.kicad_pcb (KiCad board)
At the start: 2 copper layers, 96 parts, among them J1 Conn_01x03_Pin, J2 Conn_01x04_Pin, J3 Conn_01x05, J4 Conn_01x03, U1 ADF4350, U2 ADG918BCPZ, U3 SKY66185-11, U5 AD8313xRM, U6 GRF2070, Y1 ECS-TXO-20CSMV-AC-260-AY-TR

Commit message: composants_places_pcb
Parts:
- moved C22 286.9 mm to (130.8, 102.8)
- moved C27 283.8 mm to (132.6, 107.0), turned to -90 degrees
- moved C8 282.4 mm to (126.6, 96.6), turned to -90 degrees
- moved C26 282.1 mm to (134.2, 104.4), turned to 90 degrees
- moved C28 281.9 mm to (133.8, 107.0), turned to -90 degrees
- moved C20 280.5 mm to (129.6, 101.0), turned to -90 degrees
- moved R1 278.2 mm to (120.3, 101.1), turned to -90 degrees
- moved C25 278.1 mm to (136.7, 98.1)
- moved C19 278.0 mm to (129.2, 91.2), turned to -90 degrees
- moved C21 277.5 mm to (132.0, 101.0), turned to -90 degrees
- moved C5 277.3 mm to (126.6, 99.0), turned to 90 degrees
- moved J3 277.1 mm to (123.0, 92.7)
- moved C15 276.9 mm to (134.6, 93.8)
- moved U2 276.4 mm to (130.1, 105.2), turned to 180 degrees
- moved R3 276.1 mm to (119.4, 98.6), turned to 180 degrees
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
Commit message: pcb2_pas_route
Parts:
- moved H1 81.7 mm to (123.1, 109.2)
- moved H2 76.8 mm to (108.4, 88.2)
- moved H4 42.0 mm to (146.4, 100.0)
- moved H3 36.9 mm to (143.0, 74.5)
- moved AE1 14.3 mm to (126.3, 72.7), turned to 90 degrees
Other:
- board outline added: 50.8 x 50.8 mm
Changed lines of the file:
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@@
 	(footprint "MountingHole:MountingHole_3.2mm_M3_Pad"
 		(layer "F.Cu")
-		(at 178.7 49.3)
+		(at 123.1 109.2)
 		(descr "Mounting Hole 3.2mm, M3, generated by kicad-footprint-generator mountinghole.py")
 		(tags "mountinghole M3")
@@
 	(footprint "Antenna_SMD_Wurth:AE_Wurth_WE-MCA_7488910092"
 		(layer "F.Cu")
-		(at 113 67.45 180)
+		(at 126.3 72.7 90)
 		(descr "Multilayer Chip Antenna, body 5.1x11x1.5mm, https://www.we-online.com/en/components/products/datasheet/7488910092?ki")
 		(tags "SMT, Single band")
 		(property "Reference" "AE1"
-			(at 0 -7.2 180)
+			(at 0 -7.2 90)
 			(unlocked yes)
 			(layer "F.SilkS")
@@
 		)
 		(property "Value" "Antenna"
-			(at 0 7.2 180)
+			(at 0 7.2 90)
 			(unlocked yes)
 			(layer "F.Fab")
@@
 		)
 		(property "Datasheet" "~"
-			(at 0 0 0)
+			(at 0 0 90)
 			(layer "F.Fab")
 			(hide yes)
@@
 		)
 		(property "Description" ""
-			(at 0 0 0)
+			(at 0 0 90)
 			(layer "F.Fab")
 			(hide yes)
@@
 		(attr smd)
 		(fp_line
-			(start 2.66 0.56)
-			(end 2.66 4.54)
+			(start 2.66 -4.54)
+			(end 2.66 -0.56)
 			(stroke
 				(width 0.12)
@@
 		)
 		(fp_line
-			(start 2.66 -4.54)
-			(end 2.66 -0.56)
+			(start -2.66 -4.54)
+			(end -2.66 -0.56)
 			(stroke
 				(width 0.12)
@@
 		)
 		(fp_line
-			(start -2.66 0.56)
-			(end -2.66 4.54)
+			(start 2.66 0.56)
+			(end 2.66 4.54)
 			(stroke
 				(width 0.12)
@@
 		)
 		(fp_line
-			(start -2.66 -4.54)
-			(end -2.66 -0.56)
+			(start -2.66 0.56)
+			(end -2.66 4.54)
 			(stroke
 				(width 0.12)
@@
 		)
 		(fp_text user "${REFERENCE}"
-			(at 0 0 180)
+			(at 0 0 90)
 			(unlocked yes)
 			(layer "F.Fab")
@@
 		)
 		(pad "1" smd rect
-			(at -2.1 -5.55 180)
+			(at -2.1 -5.55 90)
 			(size 1.3 1.5)
 			(layers "F.Cu" "F.Mask" "F.Paste")
 		)
 		(pad "2" smd rect
-			(at 0 -5.55 180)
+			(at 0 -5.55 90)
 			(size 1.3 1.5)
 			(layers "F.Cu" "F.Mask" "F.Paste")
@@
 		)
 		(pad "3" smd rect
-			(at 2.1 -5.55 180)
+			(at 2.1 -5.55 90)
 			(size 1.3 1.5)
 			(layers "F.Cu" "F.Mask" "F.Paste")
 		)
 		(pad "4" smd rect
-			(at -2.4 0 180)
+			(at -2.4 0 90)
 			(size 0.7 0.6)
 			(layers "F.Cu" "F.Mask" "F.Paste")
 		)
 		(pad "5" smd rect
-			(at 2.4 0 180)
+			(at 2.4 0 90)
 			(size 0.7 0.6)
 			(layers "F.Cu" "F.Mask" "F.Paste")
 		)
 		(pad "6" smd rect
-			(at -2.1 5.55 180)
+			(at -2.1 5.55 90)
 			(size 1.3 1.5)
 			(layers "F.Cu" "F.Mask" "F.Paste")
 		)
 		(pad "7" smd rect
-			(at 0 5.55 180)
+			(at 0 5.55 90)
 			(size 1.3 1.5)
 			(layers "F.Cu" "F.Mask" "F.Paste")
 		)
 		(pad "8" smd rect
-			(at 2.1 5.55 180)
+			(at 2.1 5.55 90)
 			(size 1.3 1.5)
 			(layers "F.Cu" "F.Mask" "F.Paste")
@@
 	(footprint "MountingHole:MountingHole_3.2mm_M3_Pad"
 		(layer "F.Cu")
-		(at 178.7 65.2)
+		(at 143 74.5)
 		(descr "Mounting Hole 3.2mm, M3, generated by kicad-footprint-generator mountinghole.py")
 		(tags "mountinghole M3")
@@
 	(footprint "MountingHole:MountingHole_3.2mm_M3_Pad"
 		(layer "F.Cu")
-		(at 178.7 57.25)
+		(at 108.4 88.2)
 		(descr "Mounting Hole 3.2mm, M3, generated by kicad-footprint-generator mountinghole.py")
 		(tags "mountinghole M3")
@@
 	(footprint "MountingHole:MountingHole_3.2mm_M3_Pad"
 		(layer "F.Cu")
-		(at 178.7 73.15)
+		(at 146.4 100)
 		(descr "Mounting Hole 3.2mm, M3, generated by kicad-footprint-generator mountinghole.py")
 		(tags "mountinghole M3")
@@
 		)
 	)
+	(gr_circle
+		(center 129.6 89.599798)
+		(end 129.6 64.2)
+		(stroke
+			(width 0.05)
+			(type default)
+		)
+		(fill no)
+		(layer "Edge.Cuts")
+	)
 	(embedded_fonts no)

Commit message: routage_bien_avance
Parts:
- moved H2 78.8 mm to (184.6, 68.2)
- moved H1 62.0 mm to (185.0, 105.4)
- moved H3 42.8 mm to (185.4, 80.2)
- moved H4 39.7 mm to (185.4, 92.4)
- moved J2 8.96 mm to (150.3, 92.3), turned to -90 degrees
- moved R14 1.18 mm to (139.4, 80.8), turned to 180 degrees
- moved C5 0.86 mm to (126.1, 99.7), turned to 180 degrees
- moved C19 0.70 mm to (129.2, 90.5)
- moved Y1 0.60 mm to (129.8, 88.0)
- moved C24 0.44 mm to (137.1, 100.8)
- moved C8 0.42 mm to (126.3, 96.9), turned to 90 degrees
Routing:
- net AVDD: track 0.00 -> 193.9 mm
- net GND: track 0.00 -> 51.1 mm
- net +5V: track 0.00 -> 41.9 mm
- net sig0: track 0.00 -> 24.0 mm
- net +2V5: track 0.00 -> 21.8 mm
- net Net-(U1-CPout): track 0.00 -> 20.8 mm, vias 0 -> 2
- net sig1: track 0.00 -> 16.4 mm
- net CE: track 0.00 -> 13.0 mm
- net Net-(AE1-A): track 0.00 -> 11.9 mm
- net LE: track 0.00 -> 11.1 mm
- net DATA: track 0.00 -> 9.42 mm
- net Net-(J4-Pin_1): track 0.00 -> 8.99 mm, vias 0 -> 1
- net SCK: track 0.00 -> 8.64 mm
- net Net-(J4-Pin_2): track 0.00 -> 7.71 mm
- net sig5: track 0.00 -> 6.57 mm
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- added copper zone on B.Cu, net GND
- added copper zone on F.Cu, net GND
Other:
- board size 50.8 x 50.8 mm -> 68.4 x 56 mm

Commit message: pcb2
Parts:
- C31: footprint Capacitor_SMD:C_0402_1005Metric_Pad0.74x0.62mm_HandSolder -> Capacitor_SMD:C_0603_1608Metric_Pad1.08x0.95mm_HandSolder
- L2: footprint Inductor_SMD:L_0402_1005Metric_Pad0.77x0.64mm_HandSolder -> Inductor_SMD:L_0603_1608Metric_Pad1.05x0.95mm_HandSolder
- moved C20 0.73 mm to (130.2, 101.5)
- moved C31 0.58 mm to (114.6, 100.7)
- moved L3 0.52 mm to (131.3, 100.9)
- moved C21 0.41 mm to (132.4, 100.9)
- moved L1 0.40 mm to (131.8, 99.2)
- moved L2 0.37 mm to (128.9, 99.5)
- moved C22 0.35 mm to (130.8, 103.2)
- moved U2 0.22 mm to (130.1, 105.5)
Routing:
- net GND: track 51.1 -> 117.4 mm
- net AVDD: track 193.9 -> 203.8 mm
- net sig1: track 16.4 -> 15.8 mm
- net Net-(C20-Pad2): track 2.90 -> 2.37 mm
