File: PCB1/antenne_switch/switch_antenne_pcb_projet.kicad_sch (KiCad schematic)
At the start: 10 parts, among them J1 Conn_Coaxial, J2 Conn_Coaxial

Commit message: pcb2_schematic
Parts:
- removed J1, J2: Conn_Coaxial, Connector_Coaxial:SMA_Samtec_SMA-J-P-X-ST-EM1_EdgeMount, symbol Connector:Conn_Coaxial
Connections:
- net Vers réception renamed sig3
- net Vers émission renamed sig2

Commit message: pcb2_new
Parts:
- renumbered C1 to C38, C2 to C39, L1 to L6, R1 to R11, R2 to R12, R3 to R13, U1 to U4
Changed lines of the file:
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@@
-		(color 0 0 0 0)
-	)
-	(junction
-		(at 88.9 90.17)
-		(diameter 0)
 		(color 0 0 0 0)
 	)
@@
 		(dnp no)
 		(fields_autoplaced yes)
-		(property "Reference" "#PWR02"
+		(property "Reference" "#PWR064"
 			(at 180.34 107.95 0)
 			(effects
@@
 			(project "switch_antenne_pcb_projet"
 				(path "/76074578-7479-44e4-aae5-03319eb4cd87/52934ae4-c5b0-49f4-9fc4-600729130e5d"
-					(reference "#PWR02")
+					(reference "#PWR064")
 					(unit 1)
 				)
@@
 		(dnp no)
 		(fields_autoplaced yes)
-		(property "Reference" "R2"
+		(property "Reference" "R12"
 			(at 132.08 85.725 0)
 			(effects
@@
 			(project "switch_antenne_pcb_projet"
 				(path "/76074578-7479-44e4-aae5-03319eb4cd87/52934ae4-c5b0-49f4-9fc4-600729130e5d"
-					(reference "R2")
+					(reference "R12")
 					(unit 1)
 				)
@@
 		(dnp no)
 		(fields_autoplaced yes)
-		(property "Reference" "#PWR01"
+		(property "Reference" "#PWR063"
 			(at 165.1 107.95 0)
 			(effects
@@
 			(project "switch_antenne_pcb_projet"
 				(path "/76074578-7479-44e4-aae5-03319eb4cd87/52934ae4-c5b0-49f4-9fc4-600729130e5d"
-					(reference "#PWR01")
+					(reference "#PWR063")
 					(unit 1)
 				)
@@
 		(dnp no)
 		(fields_autoplaced yes)
-		(property "Reference" "R3"
+		(property "Reference" "R13"
 			(at 142.24 85.725 0)
 			(effects
@@
 			(project "switch_antenne_pcb_projet"
 				(path "/76074578-7479-44e4-aae5-03319eb4cd87/52934ae4-c5b0-49f4-9fc4-600729130e5d"
-					(reference "R3")
+					(reference "R13")
 					(unit 1)
 				)
@@
 		(dnp no)
 		(fields_autoplaced yes)
-		(property "Reference" "U1"
+		(property "Reference" "U4"
 			(at 110.49 64.77 0)
 			(effects
@@
 			(project "switch_antenne_pcb_projet"
 				(path "/76074578-7479-44e4-aae5-03319eb4cd87/52934ae4-c5b0-49f4-9fc4-600729130e5d"
-					(reference "U1")
+					(reference "U4")
 					(unit 1)
 				)
@@
 		(on_board yes)
 		(dnp no)
-		(property "Reference" "L1"
+		(property "Reference" "L6"
 			(at 172.72 87.63 90)
 			(effects
@@
 			(project "switch_antenne_pcb_projet"
 				(path "/76074578-7479-44e4-aae5-03319eb4cd87/52934ae4-c5b0-49f4-9fc4-600729130e5d"
-					(reference "L1")
+					(reference "L6")
 					(unit 1)
 				)
@@
 		(dnp no)
 		(fields_autoplaced yes)
-		(property "Reference" "#PWR03"
+		(property "Reference" "#PWR060"
 			(at 88.9 96.52 0)
 			(effects
@@
 			(project "switch_antenne_pcb_projet"
 				(path "/76074578-7479-44e4-aae5-03319eb4cd87/52934ae4-c5b0-49f4-9fc4-600729130e5d"
-					(reference "#PWR03")
+					(reference "#PWR060")
 					(unit 1)
 				)
@@
 		(dnp no)
 		(fields_autoplaced yes)
-		(property "Reference" "#PWR05"
+		(property "Reference" "#PWR061"
 			(at 129.54 96.52 0)
 			(effects
@@
 			(project "switch_antenne_pcb_projet"
 				(path "/76074578-7479-44e4-aae5-03319eb4cd87/52934ae4-c5b0-49f4-9fc4-600729130e5d"
-					(reference "#PWR05")
+					(reference "#PWR061")
 					(unit 1)
 				)
@@
 		(dnp no)
 		(fields_autoplaced yes)
-		(property "Reference" "C1"
+		(property "Reference" "C38"
 			(at 168.91 94.615 0)
 			(effects
@@
 			(project "switch_antenne_pcb_projet"
 				(path "/76074578-7479-44e4-aae5-03319eb4cd87/52934ae4-c5b0-49f4-9fc4-600729130e5d"
-					(reference "C1")
+					(reference "C38")
 					(unit 1)
 				)
@@
 		(dnp no)
 		(fields_autoplaced yes)
-		(property "Reference" "#FLG01"
+		(property "Reference" "#FLG05"
 			(at 110.49 95.885 0)
 			(effects
@@
 			(project "switch_antenne_pcb_projet"
 				(path "/76074578-7479-44e4-aae5-03319eb4cd87/52934ae4-c5b0-49f4-9fc4-600729130e5d"
-					(reference "#FLG01")
+					(reference "#FLG05")
 					(unit 1)
 				)
@@
 		(dnp no)
 		(fields_autoplaced yes)
-		(property "Reference" "R1"
+		(property "Reference" "R11"
 			(at 91.44 85.725 0)
 			(effects
@@
 			(project "switch_antenne_pcb_projet"
 				(path "/76074578-7479-44e4-aae5-03319eb4cd87/52934ae4-c5b0-49f4-9fc4-600729130e5d"
-					(reference "R1")
+					(reference "R11")
 					(unit 1)
 				)
@@
 		(dnp no)
 		(fields_autoplaced yes)
-		(property "Reference" "#PWR06"
+		(property "Reference" "#PWR062"
 			(at 139.7 96.52 0)
 			(effects
@@
 			(project "switch_antenne_pcb_projet"
 				(path "/76074578-7479-44e4-aae5-03319eb4cd87/52934ae4-c5b0-49f4-9fc4-600729130e5d"
-					(reference "#PWR06")
+					(reference "#PWR062")
 					(unit 1)
 				)
@@
 		(dnp no)
 		(fields_autoplaced yes)
-		(property "Reference" "C2"
+		(property "Reference" "C39"
 			(at 184.15 94.615 0)
 			(effects
@@
 			(project "switch_antenne_pcb_projet"
 				(path "/76074578-7479-44e4-aae5-03319eb4cd87/52934ae4-c5b0-49f4-9fc4-600729130e5d"
-					(reference "C2")
-					(unit 1)
-				)
-			)
-		)
-	)
-	(symbol
-		(lib_id "power:PWR_FLAG")
-		(at 88.9 90.17 90)
-		(unit 1)
-		(exclude_from_sim no)
-		(in_bom yes)
-		(on_board yes)
-		(dnp no)
-		(fields_autoplaced yes)
-		(property "Reference" "#FLG02"
-			(at 86.995 90.17 0)
-			(effects
-				(font
-					(size 1.27 1.27)
-				)
-				(hide yes)
-			)
-		)
-		(property "Value" "PWR_FLAG"
-			(at 85.09 90.805 90)
-			(effects
-				(font
-					(size 1.27 1.27)
-				)
-				(justify left)
-			)
-		)
-		(property "Footprint" ""
-			(at 88.9 90.17 0)
-			(effects
-				(font
-					(size 1.27 1.27)
-				)
-				(hide yes)
-			)
-		)
-		(property "Datasheet" "~"
-			(at 88.9 90.17 0)
-			(effects
-				(font
-					(size 1.27 1.27)
-				)
-				(hide yes)
-			)
-		)
-		(property "Description" ""
-			(at 88.9 90.17 0)
-			(effects
-				(font
-					(size 1.27 1.27)
-				)
-			)
-		)
-		(pin "1"
-		)
-		(instances
-			(project "switch_antenne_pcb_projet"
-				(path "/466e3751-f273-4ede-b9d8-d94bb943d431"
-					(reference "#FLG02")
-					(unit 1)
-				)
-			)
-			(project "switch_antenne_pcb_projet"
-				(path "/76074578-7479-44e4-aae5-03319eb4cd87/52934ae4-c5b0-49f4-9fc4-600729130e5d"
-					(reference "#FLG02")
-					(unit 1)
-				)
+					(reference "C39")
+					(unit 1)
+				)

Commit message: schematic_pcb
Parts:
- AE1: footprint WE_MCA:AE_Wurth_WE-MCA_7488910092 -> Antenna_SMD_Wurth:AE_Wurth_WE-MCA_7488910092
Changed lines of the file:
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@@
-		)
-	)
-	(label "Vers réception"
-		(at 123.19 105.41 90)
-		(effects
-			(font
-				(size 1.27 1.27)
-			)
-			(justify left bottom)
-		)
-	)
-	(label "Vers émission"
-		(at 97.79 105.41 90)
-		(effects
-			(font
-				(size 1.27 1.27)
-			)
-			(justify left bottom)
 		)
 	)
@@
 			)
 		)
-		(property "Footprint" "WE_MCA:AE_Wurth_WE-MCA_7488910092"
+		(property "Footprint" "Antenna_SMD_Wurth:AE_Wurth_WE-MCA_7488910092"
 			(at 214.63 77.47 0)
 			(effects
